Commit message: feat(arac): Ackermann direksiyonlu gercek olcekli arac + IMU + LiDAR
Onceki arac 0.5 m boyunda, 4 tekerlekli bir govdeye diff-drive takiyordu.
On tekerlekler ne tahrikli ne direksiyonluydu: arka tekerlekler donmeye
calisirken on tekerlekler yere surtup direnc yapiyordu. Kamera 12 cm
yukseklikteydi ve 7 m genisligindeki yolda serit cizgileri goruntude
birkac piksel kaliyordu; Hough hicbir cizgi bulamiyordu.

Yeni arac:
  - gercek Ackermann kinematigi (on tekerlekler doner, arka tahrik)
  - 4.0 x 1.8 m govde, 2.5 m dingil mesafesi, 1200 kg
  - kamera 1.30 m'de, FOV 1.047 -> 1.40 (viraji cerceve icinde tutuyor)
  - IMU (100 Hz) ve on tampon LiDAR'i (+-90 derece, 60 m)
  - tekerleklerde acik mu1/mu2 surtunme katsayilari
  - atalet tensorleri geometriden hesaplaniyor (elle yuvarlanmis degil)

Dosya artik gercek xacro; launch icinde xacro ile isleniyor. Onceki
surumde .urdf.xacro adini tasidigi halde duz open() ile okunuyordu.

Launch tarafinda:
  - yollar get_package_share_directory uzerinden; '~/ros2_ws/src' sabiti
    kaldirildi, colcon install artik anlamli
  - tum dugumlere use_sim_time
  - TimerAction (3/4/5 s) yerine olay zinciri: gzserver basladiktan
    sonra spawn, spawn bittikten sonra dugumler
  - world / gui / rviz / algilama / use_sim_time launch argumanlari
  - static_transform_publisher --frame-id bicimine gecti
  - package.xml'e eksik bagimliliklar eklendi

Olcumle dogrulanan davranis:
  - hiz: 4.0 m/s komutuna 3.956 m/s
  - cmd_vel'deki angular.z YONELME HIZI DEGIL DIREKSIYON ACISI. Ayni
    0.3 rad komutu v=1.78'de 0.201 rad/s, v=5.02'de 0.438 rad/s yaw
    uretiyor; yonelme hizi olsa ikisi de 0.300 olurdu. Kontrolcu buna
    gore yazilmali.
  - yuksek hizda kinematik beklentinin %30 altinda donuyor: lastik
    kaymasi, beklenen understeer.
  - LiDAR: sag bariyer 2.85 m (hesap 2.86), sol 6.32 m (hesap 6.34)

LiDAR yerlesiminde iki tuzak cikti ve duzeltildi: tavanda 1.60 m'de
yatay tarama 0.80 m'lik bariyerlerin ustunden geciyordu (en yakin donus
53 m); 1.90 m'de ise sensor sasinin icinde kalip +-70 derecede kendi
govdesini goruyordu.

File: src/perception_pkg/urdf/otonom_arac.urdf.xacro (robot description, xacro)
@@ -1,68 +1,214 @@
 <?xml version="1.0"?>
-<robot name="otonom_arac">
-  <material name="mavi"><color rgba="0.1 0.3 0.8 1"/></material>
-  <material name="siyah"><color rgba="0.1 0.1 0.1 1"/></material>
-  <material name="gri"><color rgba="0.5 0.5 0.5 1"/></material>
+<!--
+  Otonom arac: Ackermann direksiyonlu, gercek otomobil olceginde.
+  Onceki surum 0.5 m boyunda, 4 tekerlekli bir govdeye diff-drive
+  takiyordu. On tekerlekler ne tahrikli ne direksiyonluydu; arka
+  tekerlekler donmeye calisirken on tekerlekler yere surtup direnc
+  yapiyordu. Ayrica kamera 12 cm yuksekteydi ve 7 m genisligindeki
+  yolda serit cizgileri goruntude birkac piksel kaliyordu; Hough
+  hicbir cizgi bulamiyordu.
+  Bu surum:
+    - gercek Ackermann kinematigi (on tekerlekler doner, arka tahrik)
+    - 4.0 x 1.8 m govde, 2.5 m dingil mesafesi
+    - kamera 1.30 m'de (on cam hizasi)
+    - IMU + 2D LiDAR
+    - tekerleklerde acik surtunme katsayilari
+  Dosya gercek xacro'dur; launch icinde xacro ile islenmelidir
+  (duz open() ile okunursa ${...} ifadeleri cozulmez).
+-->
+<robot name="otonom_arac" xmlns:xacro="http://www.ros.org/wiki/xacro">
+  <!-- ====================== PARAMETRELER ====================== -->
+  <xacro:property name="govde_uzun"  value="4.00"/>
+  <xacro:property name="govde_en"    value="1.80"/>
+  <xacro:property name="govde_yuk"   value="0.80"/>
+  <xacro:property name="govde_kutle" value="1200.0"/>
+  <xacro:property name="dingil_mesafe" value="2.50"/>  <!-- on-arka aks -->
+  <xacro:property name="iz_genislik"   value="1.60"/>  <!-- sol-sag teker -->
+  <xacro:property name="teker_yaricap" value="0.33"/>
+  <xacro:property name="teker_kalin"   value="0.25"/>
+  <xacro:property name="teker_kutle"   value="20.0"/>
+  <xacro:property name="direksiyon_kutle" value="5.0"/>
+  <xacro:property name="maks_direksiyon"  value="0.60"/>  <!-- rad, ~34 derece -->
+  <!-- Sensor yerlesimi: base_link aks hizasindadir, yani yerden
+       teker_yaricap kadar yuksektedir. Yerden istenen yukseklige
+       ulasmak icin aradaki fark dusulur. -->
+  <xacro:property name="kamera_yer_yuk" value="1.30"/>
+  <!-- LiDAR tampon hizasinda (tavanda degil). Tavanda 1.60 m'ye
+       konuldugunda yatay tarama 0.80 m'lik yol bariyerlerinin
+       USTUNDEN geciyordu: olcumde en yakin donus 53 m cikti, oysa
+       bariyer 2.3 m otedeydi. Tampon yuksekligi hem bariyeri hem
+       koni/yaya gibi alcak engelleri goruyor. -->
+  <xacro:property name="lidar_yer_yuk"  value="0.55"/>
+  <!-- Govde x in [-2.0, +2.0] arasini, z in [0.18, 0.98] arasini
+       kapliyor. LiDAR 1.90'dayken sensor sasinin ICINDE kaliyordu ve
+       +-70 derecede kendi govdesini 0.30 m'de (range_min) goruyordu.
+       Tamponun 0.10 m onune alindi. -->
+  <xacro:property name="lidar_ileri"    value="2.10"/>
+  <!-- Gorus +-90 derece ile sinirli: daha genis acilarda isinlar geriye
+       donup govdeye carpiyor. Ileri bakan otomotiv LiDAR'i zaten boyle. -->
+  <xacro:property name="lidar_aci"      value="1.5708"/>
+  <xacro:property name="kamera_ileri"   value="0.60"/>
+  <xacro:property name="kamera_egim"    value="0.10"/>  <!-- rad, asagi -->
+  <xacro:property name="PI" value="3.14159265359"/>
+  <!-- ====================== MAKROLAR ====================== -->
+  <!-- Kutu atalet tensoru -->
+  <xacro:macro name="kutu_atalet" params="m x y z">
+    <inertial>
+      <mass value="${m}"/>
+      <inertia ixx="${m*(y*y + z*z)/12.0}"
+               iyy="${m*(x*x + z*z)/12.0}"
+               izz="${m*(x*x + y*y)/12.0}"
+               ixy="0" ixz="0" iyz="0"/>
+    </inertial>
+  </xacro:macro>
+  <!-- Silindir atalet tensoru; donme ekseni z -->
+  <xacro:macro name="silindir_atalet" params="m r h">
+    <inertial>
+      <mass value="${m}"/>
+      <inertia ixx="${m*(3*r*r + h*h)/12.0}"
+               iyy="${m*(3*r*r + h*h)/12.0}"
+               izz="${m*r*r/2.0}"
+               ixy="0" ixz="0" iyz="0"/>
+    </inertial>
+  </xacro:macro>
+  <!-- Tekerlek govdesi + Gazebo surtunme ozellikleri.
+       Onceki surumde mu1/mu2 hic tanimli degildi; Gazebo varsayilani
+       kullaniliyor ve kayma ongorulemiyordu. -->
+  <xacro:macro name="tekerlek_link" params="ad">
+    <link name="${ad}">
+      <visual>
+        <origin rpy="${PI/2} 0 0"/>
+        <geometry><cylinder radius="${teker_yaricap}" length="${teker_kalin}"/></geometry>
+        <material name="lastik"/>
+      </visual>
+      <collision>
+        <origin rpy="${PI/2} 0 0"/>
+        <geometry><cylinder radius="${teker_yaricap}" length="${teker_kalin}"/></geometry>
+      </collision>
+      <xacro:silindir_atalet m="${teker_kutle}" r="${teker_yaricap}" h="${teker_kalin}"/>
+    </link>
+    <gazebo reference="${ad}">
+      <mu1>1.2</mu1>
+      <mu2>1.2</mu2>
+      <kp>1e7</kp>
+      <kd>1e3</kd>
+      <minDepth>0.002</minDepth>
+      <maxVel>10.0</maxVel>
+      <material>Gazebo/DarkGrey</material>
+    </gazebo>
+  </xacro:macro>
+  <!-- Arka tekerlek: dogrudan govdeye bagli, tahrikli -->
+  <xacro:macro name="arka_tekerlek" params="ad y_isaret">
+    <xacro:tekerlek_link ad="${ad}"/>
+    <joint name="${ad}_joint" type="continuous">
+      <parent link="base_link"/>
+      <child  link="${ad}"/>
+      <origin xyz="${-dingil_mesafe/2} ${y_isaret*iz_genislik/2} 0"/>
+      <axis xyz="0 1 0"/>
+      <limit effort="5000" velocity="100"/>
+      <dynamics damping="0.1" friction="0.1"/>
+    </joint>
+  </xacro:macro>
+  <!-- On tekerlek: once direksiyon mafsali, sonra donen tekerlek.
+       Iki kademeli olmasi Ackermann'in sarti; tek continuous mafsal
+       ile direksiyon kirilamaz. -->
+  <xacro:macro name="on_tekerlek" params="ad y_isaret">
+    <link name="${ad}_direksiyon">
+      <xacro:kutu_atalet m="${direksiyon_kutle}" x="0.1" y="0.1" z="0.1"/>
+    </link>
+    <joint name="${ad}_direksiyon_joint" type="revolute">
+      <parent link="base_link"/>
+      <child  link="${ad}_direksiyon"/>
+      <origin xyz="${dingil_mesafe/2} ${y_isaret*iz_genislik/2} 0"/>
+      <axis xyz="0 0 1"/>
+      <limit lower="${-maks_direksiyon}" upper="${maks_direksiyon}"
+             effort="20000" velocity="10"/>
+      <dynamics damping="1.0" friction="0.5"/>
+    </joint>
+    <xacro:tekerlek_link ad="${ad}"/>
+    <joint name="${ad}_joint" type="continuous">
+      <parent link="${ad}_direksiyon"/>
+      <child  link="${ad}"/>
+      <origin xyz="0 0 0"/>
+      <axis xyz="0 1 0"/>
+      <limit effort="5000" velocity="100"/>
+      <dynamics damping="0.1" friction="0.1"/>
+    </joint>
+  </xacro:macro>
+  <!-- ====================== MALZEMELER ====================== -->
+  <material name="govde_rengi"><color rgba="0.15 0.35 0.75 1"/></material>
+  <material name="lastik">     <color rgba="0.08 0.08 0.08 1"/></material>
+  <material name="cam">        <color rgba="0.2 0.25 0.3 1"/></material>
+  <material name="sensor">     <color rgba="0.6 0.6 0.62 1"/></material>
+  <!-- ====================== GOVDE ====================== -->
   <link name="base_link">
-    <visual><geometry><box size="0.5 0.3 0.15"/></geometry><material name="mavi"/></visual>
-    <collision><geometry><box size="0.5 0.3 0.15"/></geometry></collision>
-    <inertial><mass value="5.0"/>
-      <inertia ixx="0.05" iyy="0.1" izz="0.1" ixy="0" ixz="0" iyz="0"/></inertial>
-  </link>
-  <link name="tekerlek_sol_arka">
-    <visual><geometry><cylinder radius="0.07" length="0.04"/></geometry><material name="siyah"/></visual>
-    <collision><geometry><cylinder radius="0.07" length="0.04"/></geometry></collision>
-    <inertial><mass value="0.3"/>
-      <inertia ixx="0.001" iyy="0.001" izz="0.001" ixy="0" ixz="0" iyz="0"/></inertial>
-  </link>
-  <joint name="tekerlek_sol_arka_joint" type="continuous">
-    <parent link="base_link"/><child link="tekerlek_sol_arka"/>
-    <origin xyz="-0.15 0.17 -0.07" rpy="-1.5708 0 0"/><axis xyz="0 0 1"/>
-  </joint>
-  <link name="tekerlek_sag_arka">
-    <visual><geometry><cylinder radius="0.07" length="0.04"/></geometry><material name="siyah"/></visual>
-    <collision><geometry><cylinder radius="0.07" length="0.04"/></geometry></collision>
-    <inertial><mass value="0.3"/>
-      <inertia ixx="0.001" iyy="0.001" izz="0.001" ixy="0" ixz="0" iyz="0"/></inertial>
-  </link>
-  <joint name="tekerlek_sag_arka_joint" type="continuous">
-    <parent link="base_link"/><child link="tekerlek_sag_arka"/>
-    <origin xyz="-0.15 -0.17 -0.07" rpy="-1.5708 0 0"/><axis xyz="0 0 1"/>
-  </joint>
-  <link name="tekerlek_sol_on">
-    <visual><geometry><cylinder radius="0.07" length="0.04"/></geometry><material name="siyah"/></visual>
-    <collision><geometry><cylinder radius="0.07" length="0.04"/></geometry></collision>
-    <inertial><mass value="0.3"/>
-      <inertia ixx="0.001" iyy="0.001" izz="0.001" ixy="0" ixz="0" iyz="0"/></inertial>
-  </link>
-  <joint name="tekerlek_sol_on_joint" type="continuous">
-    <parent link="base_link"/><child link="tekerlek_sol_on"/>
-    <origin xyz="0.15 0.17 -0.07" rpy="-1.5708 0 0"/><axis xyz="0 0 1"/>
-  </joint>
-  <link name="tekerlek_sag_on">
-    <visual><geometry><cylinder radius="0.07" length="0.04"/></geometry><material name="siyah"/></visual>
-    <collision><geometry><cylinder radius="0.07" length="0.04"/></geometry></collision>
-    <inertial><mass value="0.3"/>
-      <inertia ixx="0.001" iyy="0.001" izz="0.001" ixy="0" ixz="0" iyz="0"/></inertial>
-  </link>
-  <joint name="tekerlek_sag_on_joint" type="continuous">
-    <parent link="base_link"/><child link="tekerlek_sag_on"/>
-    <origin xyz="0.15 -0.17 -0.07" rpy="-1.5708 0 0"/><axis xyz="0 0 1"/>
-  </joint>
+    <visual>
+      <origin xyz="0 0 ${govde_yuk/2 - 0.15}"/>
+      <geometry><box size="${govde_uzun} ${govde_en} ${govde_yuk}"/></geometry>
+      <material name="govde_rengi"/>
+    </visual>
+    <collision>
+      <origin xyz="0 0 ${govde_yuk/2 - 0.15}"/>
+      <geometry><box size="${govde_uzun} ${govde_en} ${govde_yuk}"/></geometry>
+    </collision>
+    <xacro:kutu_atalet m="${govde_kutle}"
+                       x="${govde_uzun}" y="${govde_en}" z="${govde_yuk}"/>
+  </link>
+  <gazebo reference="base_link"><material>Gazebo/Blue</material></gazebo>
+  <!-- Kabin: sadece gorsel, aracin yonunu gozle ayirt etmek icin -->
+  <link name="kabin">
+    <visual>
+      <geometry><box size="1.8 1.65 0.6"/></geometry>
+      <material name="cam"/>
+    </visual>
+    <!-- Sadece gorsel olsa da atalet sart: Gazebo ataleti olmayan
+         link'i sifir kutleli sayip uyari veriyor. -->
+    <xacro:kutu_atalet m="80.0" x="1.8" y="1.65" z="0.6"/>
+  </link>
+  <joint name="kabin_joint" type="fixed">
+    <parent link="base_link"/>
+    <child  link="kabin"/>
+    <origin xyz="-0.2 0 ${govde_yuk - 0.15 + 0.15}"/>
+  </joint>
+  <gazebo reference="kabin"><material>Gazebo/SkyBlue</material></gazebo>
+  <!-- ====================== TEKERLEKLER ====================== -->
+  <xacro:arka_tekerlek ad="arka_sol"  y_isaret="1"/>
+  <xacro:arka_tekerlek ad="arka_sag"  y_isaret="-1"/>
+  <xacro:on_tekerlek   ad="on_sol"    y_isaret="1"/>
+  <xacro:on_tekerlek   ad="on_sag"    y_isaret="-1"/>
+  <!-- Kabin ici direksiyon simidi. Gorsel olarak onemsiz ama
+       ackermann_drive plugini <steering_wheel_joint> bekliyor. -->
+  <link name="direksiyon_simidi">
+    <xacro:silindir_atalet m="1.0" r="0.18" h="0.05"/>
+  </link>
+  <joint name="direksiyon_simidi_joint" type="revolute">
+    <parent link="base_link"/>
+    <child  link="direksiyon_simidi"/>
+    <origin xyz="0.3 0.35 0.9" rpy="0 1.2 0"/>
+    <axis xyz="0 0 1"/>
+    <limit lower="-7.85" upper="7.85" effort="100" velocity="50"/>
+  </joint>
+  <!-- ====================== KAMERA ====================== -->
   <link name="kamera_link">
-    <visual><geometry><box size="0.05 0.05 0.05"/></geometry><material name="gri"/></visual>
-    <inertial><mass value="0.1"/>
-      <inertia ixx="0.0001" iyy="0.0001" izz="0.0001" ixy="0" ixz="0" iyz="0"/></inertial>
+    <visual>
+      <geometry><box size="0.08 0.12 0.06"/></geometry>
+      <material name="sensor"/>
+    </visual>
+    <xacro:kutu_atalet m="0.5" x="0.08" y="0.12" z="0.06"/>
   </link>
   <joint name="kamera_joint" type="fixed">
-    <parent link="base_link"/><child link="kamera_link"/>
-    <origin xyz="0.25 0 0.12" rpy="0 0.2 0"/>
+    <parent link="base_link"/>
+    <child  link="kamera_link"/>
+    <origin xyz="${kamera_ileri} 0 ${kamera_yer_yuk - teker_yaricap}"
+            rpy="0 ${kamera_egim} 0"/>
   </joint>
   <gazebo reference="kamera_link">
     <sensor name="arac_kamerasi" type="camera">
       <camera>
-        <horizontal_fov>1.047</horizontal_fov>
+        <!-- FOV 1.047 (60 derece) idi; 1.40 (80 derece) serit
+             cizgilerini viraj icinde de cerceve icinde tutuyor -->
+        <horizontal_fov>1.40</horizontal_fov>
         <image><width>640</width><height>480</height><format>R8G8B8</format></image>
-        <clip><near>0.1</near><far>50.0</far></clip>
+        <clip><near>0.1</near><far>150.0</far></clip>
       </camera>
       <always_on>true</always_on>
@@ -75,20 +221,115 @@
     </sensor>
   </gazebo>
+  <!-- ====================== IMU ====================== -->
+  <link name="imu_link">
+    <xacro:kutu_atalet m="0.1" x="0.04" y="0.04" z="0.02"/>
+  </link>
+  <joint name="imu_joint" type="fixed">
+    <parent link="base_link"/>
+    <child  link="imu_link"/>
+    <origin xyz="0 0 0.1"/>
+  </joint>
+  <gazebo reference="imu_link">
+    <sensor name="arac_imu" type="imu">
+      <always_on>true</always_on>
+      <update_rate>100</update_rate>
+      <imu>
+        <angular_velocity>
+          <x><noise type="gaussian"><mean>0.0</mean><stddev>2e-4</stddev></noise></x>
+          <y><noise type="gaussian"><mean>0.0</mean><stddev>2e-4</stddev></noise></y>
+          <z><noise type="gaussian"><mean>0.0</mean><stddev>2e-4</stddev></noise></z>
+        </angular_velocity>
+        <linear_acceleration>
+          <x><noise type="gaussian"><mean>0.0</mean><stddev>1.7e-2</stddev></noise></x>
+          <y><noise type="gaussian"><mean>0.0</mean><stddev>1.7e-2</stddev></noise></y>
+          <z><noise type="gaussian"><mean>0.0</mean><stddev>1.7e-2</stddev></noise></z>
+        </linear_acceleration>
+      </imu>
+      <plugin name="arac_imu_driver" filename="libgazebo_ros_imu_sensor.so">
+        <ros>
+          <namespace>arac</namespace>
+          <remapping>~/out:=imu</remapping>
+        </ros>
+        <frame_name>imu_link</frame_name>
+      </plugin>
+    </sensor>
+  </gazebo>
+  <!-- ====================== 2D LIDAR ====================== -->
+  <link name="lidar_link">
+    <visual>
+      <geometry><cylinder radius="0.05" length="0.07"/></geometry>
+      <material name="sensor"/>
+    </visual>
+    <xacro:silindir_atalet m="0.8" r="0.05" h="0.07"/>
+  </link>
+  <joint name="lidar_joint" type="fixed">
+    <parent link="base_link"/>
+    <child  link="lidar_link"/>
+    <origin xyz="${lidar_ileri} 0 ${lidar_yer_yuk - teker_yaricap}"/>
+  </joint>
+  <gazebo reference="lidar_link">
+    <sensor name="arac_lidar" type="ray">
+      <always_on>true</always_on>
+      <update_rate>15</update_rate>
+      <visualize>false</visualize>
+      <ray>
+        <scan>
+          <horizontal>
+            <samples>540</samples>
+            <resolution>1</resolution>
+            <min_angle>${-lidar_aci}</min_angle>
+            <max_angle>${lidar_aci}</max_angle>
+          </horizontal>
+        </scan>
+        <range>
+          <min>0.3</min>
+          <max>60.0</max>
+          <resolution>0.02</resolution>
+        </range>
+        <noise><type>gaussian</type><mean>0.0</mean><stddev>0.01</stddev></noise>
+      </ray>
+      <plugin name="arac_lidar_driver" filename="libgazebo_ros_ray_sensor.so">
+        <ros>
+          <namespace>arac</namespace>
+          <remapping>~/out:=scan</remapping>
+        </ros>
+        <output_type>sensor_msgs/LaserScan</output_type>
+        <frame_name>lidar_link</frame_name>
+      </plugin>
+    </sensor>
+  </gazebo>
+  <!-- ====================== SURUS ====================== -->
   <gazebo>
-    <plugin name="diff_drive" filename="libgazebo_ros_diff_drive.so">
+    <plugin name="ackermann_surus" filename="libgazebo_ros_ackermann_drive.so">
       <ros>
         <namespace>arac</namespace>
         <remapping>cmd_vel:=cmd_vel</remapping>
         <remapping>odom:=odom</remapping>
+        <remapping>distance:=mesafe</remapping>
       </ros>
-      <left_joint>tekerlek_sol_arka_joint</left_joint>
-      <right_joint>tekerlek_sag_arka_joint</right_joint>
-      <wheel_separation>0.34</wheel_separation>
-      <wheel_diameter>0.14</wheel_diameter>
-      <max_wheel_torque>20</max_wheel_torque>
-      <max_wheel_acceleration>1.0</max_wheel_acceleration>
+      <update_rate>100.0</update_rate>
+      <front_left_joint>on_sol_joint</front_left_joint>
+      <front_right_joint>on_sag_joint</front_right_joint>
+      <rear_left_joint>arka_sol_joint</rear_left_joint>
+      <rear_right_joint>arka_sag_joint</rear_right_joint>
+      <left_steering_joint>on_sol_direksiyon_joint</left_steering_joint>
+      <right_steering_joint>on_sag_direksiyon_joint</right_steering_joint>
+      <steering_wheel_joint>direksiyon_simidi_joint</steering_wheel_joint>
+      <max_steer>${maks_direksiyon}</max_steer>
+      <max_steering_angle>7.85</max_steering_angle>
+      <max_speed>20.0</max_speed>
+      <!-- 1200 kg'lik bir govde icin kazanclar demo degerlerinin
+           cok uzerinde olmali; dusuk kazancla direksiyon komutu
+           takip edemiyor. -->
+      <left_steering_pid_gain>20000 0 2000</left_steering_pid_gain>
+      <left_steering_i_range>0 0</left_steering_i_range>
+      <right_steering_pid_gain>20000 0 2000</right_steering_pid_gain>
+      <right_steering_i_range>0 0</right_steering_i_range>
+      <linear_velocity_pid_gain>5000 0 200</linear_velocity_pid_gain>
+      <linear_velocity_i_range>0 0</linear_velocity_i_range>
       <publish_odom>true</publish_odom>
       <publish_odom_tf>true</publish_odom_tf>
-      <publish_wheel_tf>false</publish_wheel_tf>
+      <publish_wheel_tf>true</publish_wheel_tf>
+      <publish_distance>true</publish_distance>
       <odometry_frame>odom</odometry_frame>
       <robot_base_frame>base_link</robot_base_frame>
