Commit message: feat(serit): HSV + kus bakisi (IPM) + saf takip ile serit takibi
Onceki surum serit takip ETMIYORDU. Olcum: Canny/Hough ham goruntude
tek bir cizgi bile bulamiyor, iki liste de bos kalinca sol_x=0 /
sag_x=640 oluyor, serit merkezi tam goruntu merkezine dusuyor ve hata
SIFIR cikiyordu. Araç tam gazda duz gidiyor, ilk virajda dis bariyere
yapisiyordu (x=43'te takili kalmisti).

Yeni boru hatti:
  - Renk maskeleri: sari = orta cizgi, beyaz = kenar. Siniflandirma
    egim tahminine degil renge dayaniyor; virajda bozulmuyor.
  - IPM: homografi 4 nokta elle secilerek degil, kameranin ic/dis
    parametrelerinden analitik turetiliyor (yeni perception_pkg/ipm.py).
    Gidis-donus hatasi 7.6e-15 m.
  - Saf takip (pure pursuit) DOGRUDAN DIREKSIYON ACISI uretiyor; olcumle
    dogrulanan eklenti semantigi bu.
  - Egrilige gore hiz, serit kaybinda yavasla/dur, sensor QoS.

Yol boyunca bulunan iki donanim hatasi:
  1. Kamera 0.60 m'de iken govdenin on ust kosesi goruntude v=288
     satirina dusuyor, altindaki 192 satiri (karenin %40'i) kaputla
     dolduruyordu; yolun ilk 6.4 m'si kordu. Kamera on tampona (1.95 m)
     alindi, gorus 3.6 m'den basliyor.
  2. Dunyada IKI beyaz cizgi var (dis kenar -1.75, ic kenar +5.25) ama
     TEK sari. Kayan pencere ic kenara kilitlenip serit merkezini 3.5 m
     kaydirmis, araci kars'i seride surmustu (y=-22.1, olmasi gereken
     -26.75). Beyazin beklentisi artik sari gorundugu her karede ona
     gore tohumlaniyor; ayrica sari-beyaz ayrimi bir serit genisligine
     uymazsa sariya guveniliyor.

Olculen ilerleme (165 s kosu):
  once          : 39 m, sapma ort 1.64 m, ilk virajda pistten cikti
  kamera duzeldi: 227 m (0.82 tur), sapma ort 0.64 m, seritte kaldi
  bu commit     : 398 m (1.44 TUR), ort 2.85 m/s

Kalan is: saf takibin virajda biraktigi kalici yanal offset. Araç turu
tamamliyor ama seridin ortasi yerine sari cizgiye yaslanarak gidiyor
(sapma ort 1.63 m). Ortalanma ayari ve hiz profili ayarlanmali.

File: src/perception_pkg/urdf/otonom_arac.urdf.xacro (robot description, xacro)
@@ -34,4 +34,12 @@
        ulasmak icin aradaki fark dusulur. -->
   <xacro:property name="kamera_yer_yuk" value="1.30"/>
+  <!-- Kamera kaputun ONUNDE olmak zorunda. 0.60 m'de (on cam hizasi)
+       iken govdenin on ust kosesi (x=2.0, z=0.98) goruntude v=288
+       satirina dusuyor ve altindaki 192 satiri (karenin %40'i)
+       kaputla dolduruyordu; yolun ilk 6.4 m'si kor kaliyordu.
+       Kamerayi yerinde tutup kaputu FOV disina cikarmak icin kaputun
+       0.20 m'ye inmesi gerekirdi. Bunun yerine kamera on tampona
+       alindi; gorus artik 3.6 m'den basliyor. -->
+  <xacro:property name="kamera_ileri"   value="1.95"/>
   <!-- LiDAR tampon hizasinda (tavanda degil). Tavanda 1.60 m'ye
        konuldugunda yatay tarama 0.80 m'lik yol bariyerlerinin
@@ -48,5 +56,4 @@
        donup govdeye carpiyor. Ileri bakan otomotiv LiDAR'i zaten boyle. -->
   <xacro:property name="lidar_aci"      value="1.5708"/>
-  <xacro:property name="kamera_ileri"   value="0.60"/>
   <xacro:property name="kamera_egim"    value="0.10"/>  <!-- rad, asagi -->
   <xacro:property name="PI" value="3.14159265359"/>
